Commit message: gemini mount

File: turtlebot4_description/urdf/standard/turtlebot4.urdf.xacro (robot description, xacro)
@@ -30,4 +30,7 @@
   <xacro:property name="camera_mount_y_offset"         value="${0*cm2m}"/>
   <xacro:property name="camera_mount_z_offset"         value="${5.257*cm2m}"/>
+  <xacro:property name="gemini_mount_x_offset"         value="${-7*cm2m}"/>
+  <xacro:property name="gemini_mount_y_offset"         value="${6.5*cm2m}"/>
+  <xacro:property name="gemini_mount_z_offset"         value="${13.5*cm2m}"/>
   <xacro:property name="oakd_pro_x_offset"             value="${5.84*cm2m}"/>
   <xacro:property name="oakd_pro_y_offset"             value="${0*cm2m}"/>
@@ -95,10 +98,10 @@
             rpy="0 0 ${pi/2}"/>
   </xacro:rplidar>
-  <xacro:camera_bracket name="oakd_camera_bracket">
+  <!--<xacro:camera_bracket name="oakd_camera_bracket">
     <origin xyz="${camera_mount_x_offset} ${camera_mount_y_offset} ${camera_mount_z_offset}"/>
   </xacro:camera_bracket>
   <xacro:oakd model="pro" parent_link="oakd_camera_bracket">
     <origin xyz="${oakd_pro_x_offset} ${oakd_pro_y_offset} ${oakd_pro_z_offset}"/>
-  </xacro:oakd>
+  </xacro:oakd>-->
   <!-- Base footprint for navigation -->
   <link name="base_footprint" />
@@ -109,3 +112,9 @@
     <child link="base_footprint" />
   </joint>
+  <link name="gemini_link" />
+  <joint name="gemini_link_joint" type="fixed">
+    <origin xyz="${gemini_mount_x_offset} ${gemini_mount_y_offset} ${gemini_mount_z_offset}" rpy="0 0 0" />
+    <parent link="shell_link" />
+    <child link="gemini_link" />
+  </joint>
 </robot>
